File: Clock/NixieClock.kicad_pcb (KiCad board)
At the start: 2 copper layers, 130.8 x 114.9 mm, 58 parts, among them J1 PJ-079BH, J2 Conn_02x10_Top_Bottom, J3 Conn_02x10_Top_Bottom, J4 Conn_02x10_Top_Bottom, J5 Conn_02x10_Odd_Even, J6 Conn_02x10_Odd_Even, J7 Conn_02x10_Odd_Even, Q1 2N2097, Q2 SI2333DDS-T1-GE3, Q3 T2N7002AK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

Commit message: Add v2.0 plots
Parts:
- removed C8: 4.7u, Capacitor_SMD:C_0603_1608Metric_Pad1.05x0.95mm_HandSolder
- removed R5: 115k, Resistor_SMD:R_0603_1608Metric_Pad1.05x0.95mm_HandSolder
- removed R6: 25.5k, Resistor_SMD:R_0603_1608Metric_Pad1.05x0.95mm_HandSolder
- removed the REF** at (164.0, 161.5)
- removed the REF** at (164.0, 109.3)
- removed the REF** at (38.2, 161.5)
- removed the REF** at (38.2, 109.3)
- added D6: BZX84Cxx, Diode_SMD:D_SOT-23_ANK, F.Cu at (93.8, 159.0)
- added Q5: SI2343DS, Package_TO_SOT_SMD:SOT-23_Handsoldering, F.Cu at (90.0, 135.5)
- added REF**: MountingHole_3.2mm_M3, MountingHole:MountingHole_3.2mm_M3, F.Cu at (39.2, 170.5)
- added REF**: MountingHole_3.2mm_M3, MountingHole:MountingHole_3.2mm_M3, F.Cu at (39.2, 120.2)
- added REF**: MountingHole_3.2mm_M3, MountingHole:MountingHole_3.2mm_M3, F.Cu at (163.0, 120.2)
- added REF**: MountingHole_3.2mm_M3, MountingHole:MountingHole_3.2mm_M3, F.Cu at (163.0, 170.5)
- added SYM1: SYM_Flash_Small, Clock:HighVoltage, F.Cu at (48.0, 169.0)
- C1: value 220u -> 330u
- C5: value 33p -> 10u; footprint Capacitor_SMD:C_0603_1608Metric_Pad1.05x0.95mm_HandSolder -> Capacitor_SMD:C_0805_2012Metric_Pad1.15x1.40mm_HandSolder
- C6: value 10u -> 22u; footprint Capacitor_SMD:C_1210_3225Metric_Pad1.42x2.65mm_HandSolder -> Capacitor_SMD:C_0805_2012Metric_Pad1.15x1.40mm_HandSolder
- C7: footprint Capacitor_SMD:C_1210_3225Metric_Pad1.42x2.65mm_HandSolder -> Capacitor_SMD:C_0805_2012Metric_Pad1.15x1.40mm_HandSolder
- Q1: value 2N2097 -> 2N2907
- Q2: value SI2333DDS-T1-GE3 -> SI2343DS
- R10, R11, R8, R9: value 22k -> 33.2k
- R12: value 20 -> 22
- R14: value 115k -> 499k
- R7: value 680 -> 2k
- U5: value AP65251 -> AP63203; footprint Package_TO_SOT_SMD:TSOT-23-6_HandSoldering -> Package_TO_SOT_SMD:TSOT-23-6
- moved C5 21.4 mm to (70.0, 165.5), turned to 270 degrees
- moved C4 18.3 mm to (79.5, 165.5), turned to 270 degrees
- moved C1 14.7 mm to (63.0, 138.0), turned to 90 degrees
- moved U5 13.6 mm to (74.5, 165.5)
- moved C2 11.9 mm to (53.5, 160.5), turned to 90 degrees
- moved Q1 11.3 mm to (60.0, 153.5)
- moved C6 11.3 mm to (86.0, 159.0), turned to 270 degrees
- moved C7 10.8 mm to (89.5, 159.0), turned to 270 degrees
- moved R1 10.0 mm to (52.8, 136.4)
- moved C3 10.0 mm to (50.3, 147.3)
- moved C9 10.0 mm to (43.5, 151.5)
- moved D1 10.0 mm to (61.7, 158.7)
- moved D2 10.0 mm to (61.7, 147.3)
- moved D5 10.0 mm to (39.0, 144.5)
- moved F1 10.0 mm to (39.0, 149.5)
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Connections:
- net Net-(Q2-Pad1) renamed T_ON
- C5 pad 1: +3.3V -> +12V
- C5 pad 2: Net-(C5-Pad2) -> GND
- C6 pad 1: +12V -> +3.3V
- J2 pad 2: Net-(J2-Pad2) -> +170V
- J2 pad 6: Net-(J2-Pad6) -> +12V
- J5 pad 15: Net-(J5-Pad15) -> +12V
- J5 pad 19: Net-(J5-Pad19) -> +170V
- L1 pad 1: Net-(C1-Pad1) -> Net-(L1-Pad1)
- Q1 pad 1: Net-(D2-Pad1) -> Net-(D2-Pad2)
- Q1 pad 2: Net-(D2-Pad2) -> Net-(D2-Pad1)
- Q4 pad 1: Net-(C9-Pad1) -> +12V_UNSAFE
- Q4 pad 2: +12V_UNSAFE -> Net-(C9-Pad1)
- U5 pad 1: Net-(C4-Pad1) -> +3.3V
- U5 pad 2: GND -> +12V
- U5 pad 3: Net-(C5-Pad2) -> +12V
- U5 pad 4: +12V -> GND
- U5 pad 5: +12V -> Net-(C4-Pad2)
- U5 pad 6: Net-(C4-Pad2) -> Net-(C4-Pad1)
Routing:
- net T_ON: track 14.3 -> 58.5 mm, vias 2 -> 4
- net L3_8: track 157.2 -> 121.3 mm, vias 2 -> 1
- net L3_7: track 153.1 -> 122.7 mm
- net L1_7: track 125.0 -> 97.1 mm, vias 0 -> 2
- net +12V: track 262.5 -> 236.0 mm
- net L1_6: track 115.7 -> 96.0 mm, vias 0 -> 3
- net L1_8: track 87.4 -> 103.7 mm, vias 2 -> 3
- net L3_6: track 141.2 -> 125.4 mm
- net L1_9: track 87.3 -> 102.9 mm, vias 2 -> 3
- net Net-(C5-Pad2): track 15.0 -> 0.00 mm
- net Net-(C1-Pad1): track 65.6 -> 50.8 mm
- net Net-(L1-Pad1): track 0.00 -> 13.8 mm
- net L2_4: track 88.3 -> 101.5 mm, vias 2 -> 3
- net L3_4: track 107.5 -> 96.3 mm, vias 1 -> 3
- net L3_1: track 68.2 -> 57.7 mm, vias 1 -> 3
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Other:
- board size 130.8 x 114.9 mm -> 130.8 x 116.9 mm
- board text added: "DANGER HIGH VOLTAGE"
- board text removed: "v2.0"

Commit message: Remove a "fast-discharge" transistor, as it was not operating as intended due to emitter-base breakdown. It was pretty much optional anyway.
Parts:
- removed Q4: 2N3906, Package_TO_SOT_SMD:SOT-23_Handsoldering
Changed lines of the file:
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@@
-(kicad_pcb (version 20171130) (host pcbnew 5.1.4)
+(kicad_pcb (version 20171130) (host pcbnew 5.1.5)
   (general
     (thickness 1.6)
@@
     (tracks 1249)
     (zones 0)
-    (modules 58)
+    (modules 57)
     (nets 127)
   )
@@
     (add_net L4_9)
   )
+  (module Clock:PJ079BH (layer F.Cu)
+    (at 45.847 127.237 270)
+    (descr PJ-079BH-1)
+    (tags Connector)
+    (fp_text reference J1 (at -4.35 -4.55 90) (layer F.SilkS)
+      (effects (font (size 1.27 1.27) (thickness 0.254)))
+    )
+    (fp_text value PJ-079BH (at -4.35 -4.55 90) (layer F.SilkS) hide
+      (effects (font (size 1.27 1.27) (thickness 0.254)))
+    )
+    (fp_text user %R (at -4.35 -4.55 90) (layer F.Fab)
+      (effects (font (size 1.27 1.27) (thickness 0.254)))
+    )
+    (fp_line (start -10.3 -9.6) (end 1.2 -9.6) (layer F.Fab) (width 0.2))
+    (fp_line (start 1.2 -9.6) (end 1.2 0.5) (layer F.Fab) (width 0.2))
+    (fp_line (start 1.2 0.5) (end -10.3 0.5) (layer F.Fab) (width 0.2))
+    (fp_line (start -10.3 0.5) (end -10.3 -9.6) (layer F.Fab) (width 0.2))
+    (fp_line (start -11.3 -12.326) (end 2.6 -12.326) (layer F.CrtYd) (width 0.1))
+    (fp_line (start 2.6 -12.326) (end 2.6 3.226) (layer F.CrtYd) (width 0.1))
+    (fp_line (start 2.6 3.226) (end -11.3 3.226) (layer F.CrtYd) (width 0.1))
+    (fp_line (start -11.3 3.226) (end -11.3 -12.326) (layer F.CrtYd) (width 0.1))
+    (fp_line (start -9.3 -9.6) (end -10.3 -9.6) (layer F.SilkS) (width 0.1))
+    (fp_line (start -10.3 -9.6) (end -10.3 0.5) (layer F.SilkS) (width 0.1))
+    (fp_line (start -10.3 0.5) (end -9.3 0.5) (layer F.SilkS) (width 0.1))
+    (fp_line (start -0.1 2.2) (end -0.1 2.2) (layer F.SilkS) (width 0.2))
+    (fp_line (start 0.1 2.2) (end 0.1 2.2) (layer F.SilkS) (width 0.2))
+    (fp_arc (start 0 2.2) (end -0.1 2.2) (angle -180) (layer F.SilkS) (width 0.2))
+    (fp_arc (start 0 2.2) (end 0.1 2.2) (angle -180) (layer F.SilkS) (width 0.2))
+    (pad 1 thru_hole oval (at 0 0 270) (size 2.7 1.5) (drill oval 2 0.8) (layers *.Cu *.Mask)
+      (net 87 +12V_UNSAFE))
+    (pad 2 thru_hole oval (at 0 -8.6 270) (size 2.7 1.5) (drill oval 2 0.8) (layers *.Cu *.Mask)
+      (net 1 GND))
+    (pad 3 thru_hole oval (at 0 -3.4 270) (size 2.7 1.5) (drill oval 2 0.8) (layers *.Cu *.Mask)
+      (net 1 GND))
+    (pad MH1 thru_hole oval (at -7.3 -9.5 270) (size 3 1.5) (drill oval 2.3 0.8) (layers *.Cu *.Mask)
+      (net 1 GND))
+    (pad MH2 thru_hole oval (at -7.3 0.4 270) (size 3 1.5) (drill oval 2.3 0.8) (layers *.Cu *.Mask)
+      (net 1 GND))
+    (pad MH3 np_thru_hole circle (at -6.3 -3.3 270) (size 2.6 0) (drill 2.6) (layers *.Cu *.Mask))
+  )
   (module Resistor_SMD:R_0603_1608Metric_Pad1.05x0.95mm_HandSolder (layer F.Cu)
     (at 61.722 143.477 180)
@@
     )
   )
-  (module Clock:PJ079BH (layer F.Cu)
-    (at 45.847 127.237 270)
-    (descr PJ-079BH-1)
-    (tags Connector)
-    (fp_text reference J1 (at -3.737 -4.653 180) (layer F.SilkS)
-      (effects (font (size 1.27 1.27) (thickness 0.254)))
-    )
-    (fp_text value PJ-079BH (at -4.35 -4.55 90) (layer F.SilkS) hide
-      (effects (font (size 1.27 1.27) (thickness 0.254)))
-    )
-    (fp_arc (start 0 2.2) (end 0.1 2.2) (angle -180) (layer F.SilkS) (width 0.2))
-    (fp_arc (start 0 2.2) (end -0.1 2.2) (angle -180) (layer F.SilkS) (width 0.2))
-    (fp_line (start 0.1 2.2) (end 0.1 2.2) (layer F.SilkS) (width 0.2))
-    (fp_line (start -0.1 2.2) (end -0.1 2.2) (layer F.SilkS) (width 0.2))
-    (fp_line (start -10.3 0.5) (end -9.3 0.5) (layer F.SilkS) (width 0.1))
-    (fp_line (start -10.3 -9.6) (end -10.3 0.5) (layer F.SilkS) (width 0.1))
-    (fp_line (start -9.3 -9.6) (end -10.3 -9.6) (layer F.SilkS) (width 0.1))
-    (fp_line (start -11.3 3.226) (end -11.3 -12.326) (layer F.CrtYd) (width 0.1))
-    (fp_line (start 2.6 3.226) (end -11.3 3.226) (layer F.CrtYd) (width 0.1))
-    (fp_line (start 2.6 -12.326) (end 2.6 3.226) (layer F.CrtYd) (width 0.1))
-    (fp_line (start -11.3 -12.326) (end 2.6 -12.326) (layer F.CrtYd) (width 0.1))
-    (fp_line (start -10.3 0.5) (end -10.3 -9.6) (layer F.Fab) (width 0.2))
-    (fp_line (start 1.2 0.5) (end -10.3 0.5) (layer F.Fab) (width 0.2))
-    (fp_line (start 1.2 -9.6) (end 1.2 0.5) (layer F.Fab) (width 0.2))
-    (fp_line (start -10.3 -9.6) (end 1.2 -9.6) (layer F.Fab) (width 0.2))
-    (fp_text user %R (at -4.35 -4.55 90) (layer F.Fab)
-      (effects (font (size 1.27 1.27) (thickness 0.254)))
-    )
-    (pad MH3 np_thru_hole circle (at -6.3 -3.3 270) (size 2.6 0) (drill 2.6) (layers *.Cu *.Mask))
-    (pad MH2 thru_hole oval (at -7.3 0.4 270) (size 3 1.5) (drill oval 2.3 0.8) (layers *.Cu *.Mask)
-      (net 1 GND))
-    (pad MH1 thru_hole oval (at -7.3 -9.5 270) (size 3 1.5) (drill oval 2.3 0.8) (layers *.Cu *.Mask)
-      (net 1 GND))
-    (pad 3 thru_hole oval (at 0 -3.4 270) (size 2.7 1.5) (drill oval 2 0.8) (layers *.Cu *.Mask)
-      (net 1 GND))
-    (pad 2 thru_hole oval (at 0 -8.6 270) (size 2.7 1.5) (drill oval 2 0.8) (layers *.Cu *.Mask)
-      (net 1 GND))
-    (pad 1 thru_hole oval (at 0 0 270) (size 2.7 1.5) (drill oval 2 0.8) (layers *.Cu *.Mask)
-      (net 87 +12V_UNSAFE))
-  )
   (module Capacitor_SMD:C_0805_2012Metric_Pad1.15x1.40mm_HandSolder (layer F.Cu)
     (at 86 159 270)
@@
     )
   )
-  (module Package_TO_SOT_SMD:SOT-23_Handsoldering (layer F.Cu)
-    (at 44.5 147)
-    (descr "SOT-23, Handsoldering")
-    (tags SOT-23)
-    (attr smd)
-    (fp_text reference Q4 (at 0 -2.5) (layer F.SilkS)
-      (effects (font (size 1 1) (thickness 0.15)))
-    )
-    (fp_text value 2N3906 (at 0 2.5) (layer F.Fab)
-      (effects (font (size 1 1) (thickness 0.15)))
-    )
-    (fp_line (start 0.76 1.58) (end -0.7 1.58) (layer F.SilkS) (width 0.12))
-    (fp_line (start -0.7 1.52) (end 0.7 1.52) (layer F.Fab) (width 0.1))
-    (fp_line (start 0.7 -1.52) (end 0.7 1.52) (layer F.Fab) (width 0.1))
-    (fp_line (start -0.7 -0.95) (end -0.15 -1.52) (layer F.Fab) (width 0.1))
-    (fp_line (start -0.15 -1.52) (end 0.7 -1.52) (layer F.Fab) (width 0.1))
-    (fp_line (start -0.7 -0.95) (end -0.7 1.5) (layer F.Fab) (width 0.1))
-    (fp_line (start 0.76 -1.58) (end -2.4 -1.58) (layer F.SilkS) (width 0.12))
-    (fp_line (start -2.7 1.75) (end -2.7 -1.75) (layer F.CrtYd) (width 0.05))
-    (fp_line (start 2.7 1.75) (end -2.7 1.75) (layer F.CrtYd) (width 0.05))
-    (fp_line (start 2.7 -1.75) (end 2.7 1.75) (layer F.CrtYd) (width 0.05))
-    (fp_line (start -2.7 -1.75) (end 2.7 -1.75) (layer F.CrtYd) (width 0.05))
-    (fp_line (start 0.76 -1.58) (end 0.76 -0.65) (layer F.SilkS) (width 0.12))
-    (fp_line (start 0.76 1.58) (end 0.76 0.65) (layer F.SilkS) (width 0.12))
-    (fp_text user %R (at 0 0 90) (layer F.Fab)
-      (effects (font (size 0.5 0.5) (thickness 0.075)))
-    )
-    (pad 3 smd rect (at 1.5 0) (size 1.9 0.8) (layers F.Cu F.Paste F.Mask)
-      (net 1 GND))
-    (pad 2 smd rect (at -1.5 0.95) (size 1.9 0.8) (layers F.Cu F.Paste F.Mask)
-      (net 122 "Net-(C9-Pad1)"))
-    (pad 1 smd rect (at -1.5 -0.95) (size 1.9 0.8) (layers F.Cu F.Paste F.Mask)
-      (net 87 +12V_UNSAFE))
-    (model ${KISYS3DMOD}/Package_TO_SOT_SMD.3dshapes/SOT-23.wrl
-      (at (xyz 0 0 0))
-      (scale (xyz 1 1 1))
-      (rotate (xyz 0 0 0))
-    )
-  )
   (module Clock:HighVoltage locked (layer F.Cu)
     (at 48 169)
@@
   (via (at 84.91 150.172) (size 0.5) (drill 0.3) (layers F.Cu B.Cu) (net 1))
   (via (at 163.83 165.575) (size 0.5) (drill 0.3) (layers F.Cu B.Cu) (net 1))
-  (via (at 73.91 171) (size 0.5) (drill 0.3) (layers F.Cu B.Cu) (net 1))
   (via (at 149.91 147.172) (size 0.5) (drill 0.3) (layers F.Cu B.Cu) (net 1))
   (via (at 135.128 131.158) (size 0.5) (drill 0.3) (layers F.Cu B.Cu) (net 1))
@@
   (via (at 51.054 145.382) (size 0.5) (drill 0.3) (layers F.Cu B.Cu) (net 1) (status 30))
   (via (at 53.91 124.172) (size 0.5) (drill 0.3) (layers F.Cu B.Cu) (net 1))
+  (via (at 73.91 171) (size 0.5) (drill 0.3) (layers F.Cu B.Cu) (net 1))
   (segment (start 55.307 141.572) (end 55.307 142.842) (width 1) (layer F.Cu) (net 2) (status 30))
   (segment (start 57.277 142.842) (end 58.68563 141.43337) (width 1) (layer F.Cu) (net 2))
